File: design/isolated_current_sensor.sch (KiCad schematic (older format))
At the start: 7 parts, among them U3 AMC1303

Commit message: Added buffer to restore signal before opamp analog filter
Signed-off-by: Marcos Chaparro <mchaparro@paltatech.com>
Connections:
- net VIN-: no longer names the net of C21.2, R10.2, U3.3 (VINN)
Changed lines of the file:
@@
 Text Notes 900  1550 0    260  ~ 52
 0-650V phase voltage measurement\nusing isolation amplifier
-Text Label 5100 4250 0    30   ~ 0
-VIN-
 Wire Wire Line
 	5100 3450 5100 3500
